File: controller_pcb/controller_pcb/controller_pcb.kicad_sch (KiCad schematic)
At the start: 26 parts, among them SW1 SW_MEC_5E, SW10 SW_MEC_5E, SW11 SW_MEC_5E, SW12 SW_MEC_5E, SW2 SW_MEC_5E, SW3 SW_MEC_5E, SW4 SW_MEC_5E, SW5 SW_MEC_5E, SW6 SW_MEC_5E, SW7 SW_MEC_5E, SW8 SW_MEC_5E, SW9 SW_MEC_5E

Commit message: didnt save
Parts:
- added U?: COM-09032, XDCR_COM-09032, symbol COM-09032:COM-09032
Connections:
- net +3V3: now also U?.H1 (H+), U?.V1 (V+)
- net GND: now also U?.H3 (H-), U?.V3 (V-)
- new net: U?.S1 (SHIELD), U?.S2 (SHIELD), U?.S3 (SHIELD), U?.S4 (SHIELD)
Changed lines of the file:
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@@
   (junction (at 22.86 180.34) (diameter 0) (color 0 0 0 0)
   )
+  (junction (at 254 74.93) (diameter 0) (color 0 0 0 0)
+  )
+  (junction (at 259.08 62.23) (diameter 0) (color 0 0 0 0)
+  )
   (junction (at 233.68 21.59) (diameter 0) (color 0 0 0 0)
   )
@@
     (stroke (width 0) (type default) (color 0 0 0 0))
   )
+  (wire (pts (xy 262.89 64.77) (xy 254 64.77))
+    (stroke (width 0) (type default) (color 0 0 0 0))
+  )
   (wire (pts (xy 35.56 36.83) (xy 35.56 49.53))
     (stroke (width 0) (type default) (color 0 0 0 0))
@@
     (stroke (width 0) (type default) (color 0 0 0 0))
   )
+  (wire (pts (xy 254 64.77) (xy 254 74.93))
+    (stroke (width 0) (type default) (color 0 0 0 0))
+  )
   (wire (pts (xy 260.35 33.02) (xy 260.35 36.83))
     (stroke (width 0) (type default) (color 0 0 0 0))
@@
     (stroke (width 0) (type default) (color 0 0 0 0))
   )
+  (wire (pts (xy 262.89 62.23) (xy 259.08 62.23))
+    (stroke (width 0) (type default) (color 0 0 0 0))
+  )
   (wire (pts (xy 134.62 138.43) (xy 130.81 138.43))
     (stroke (width 0) (type default) (color 0 0 0 0))
   )
+  (wire (pts (xy 259.08 62.23) (xy 259.08 57.15))
+    (stroke (width 0) (type default) (color 0 0 0 0))
+  )
   (wire (pts (xy 31.75 190.5) (xy 39.37 190.5))
     (stroke (width 0) (type default) (color 0 0 0 0))
@@
     (stroke (width 0) (type default) (color 0 0 0 0))
   )
+  (wire (pts (xy 262.89 74.93) (xy 254 74.93))
+    (stroke (width 0) (type default) (color 0 0 0 0))
+  )
   (wire (pts (xy 139.7 151.13) (xy 139.7 171.45))
     (stroke (width 0) (type default) (color 0 0 0 0))
@@
     (stroke (width 0) (type default) (color 0 0 0 0))
   )
+  (wire (pts (xy 259.08 72.39) (xy 259.08 62.23))
+    (stroke (width 0) (type default) (color 0 0 0 0))
+  )
   (wire (pts (xy 229.87 33.02) (xy 229.87 39.37))
     (stroke (width 0) (type default) (color 0 0 0 0))
@@
     (stroke (width 0) (type default) (color 0 0 0 0))
   )
+  (wire (pts (xy 254 74.93) (xy 254 90.17))
+    (stroke (width 0) (type default) (color 0 0 0 0))
+  )
   (wire (pts (xy 19.05 76.2) (xy 22.86 76.2))
     (stroke (width 0) (type default) (color 0 0 0 0))
@@
   )
   (wire (pts (xy 33.02 49.53) (xy 35.56 49.53))
+    (stroke (width 0) (type default) (color 0 0 0 0))
+  )
+  (wire (pts (xy 262.89 72.39) (xy 259.08 72.39))
     (stroke (width 0) (type default) (color 0 0 0 0))
   )
@@
     (pin "1")
     (pin "2")
+  )
+  (symbol (lib_id "power:+3.3V") (at 259.08 57.15 0) (unit 1)
+    (in_bom yes) (on_board yes) (fields_autoplaced)
+    (property "Reference" "#PWR?" (id 0) (at 259.08 60.96 0)
+      (effects (font (size 1.27 1.27)) hide)
+    )
+    (property "Value" "+3.3V" (id 1) (at 259.08 52.07 0))
+    (property "Footprint" "" (id 2) (at 259.08 57.15 0)
+      (effects (font (size 1.27 1.27)) hide)
+    )
+    (property "Datasheet" "" (id 3) (at 259.08 57.15 0)
+      (effects (font (size 1.27 1.27)) hide)
+    )
+    (pin "1")
   )
   (symbol (lib_id "Switch:SW_MEC_5E") (at 27.94 49.53 0) (unit 1)
@@
     (pin "1")
   )
+  (symbol (lib_id "power:GND") (at 254 90.17 0) (unit 1)
+    (in_bom yes) (on_board yes) (fields_autoplaced)
+    (property "Reference" "#PWR?" (id 0) (at 254 96.52 0)
+      (effects (font (size 1.27 1.27)) hide)
+    )
+    (property "Value" "GND" (id 1) (at 254 95.25 0))
+    (property "Footprint" "" (id 2) (at 254 90.17 0)
+      (effects (font (size 1.27 1.27)) hide)
+    )
+    (property "Datasheet" "" (id 3) (at 254 90.17 0)
+      (effects (font (size 1.27 1.27)) hide)
+    )
+    (pin "1")
+  )
   (symbol (lib_id "Regulator_Linear:XC6206PxxxMR") (at 247.65 21.59 0) (unit 1)
     (in_bom yes) (on_board yes) (fields_autoplaced)
@@
     (pin "2")
   )
+  (symbol (lib_id "COM-09032:COM-09032") (at 275.59 72.39 0) (unit 1)
+    (in_bom yes) (on_board yes) (fields_autoplaced)
+    (property "Reference" "U?" (id 0) (at 284.48 72.3899 0)
+      (effects (font (size 1.27 1.27)) (justify left))
+    )
+    (property "Value" "COM-09032" (id 1) (at 284.48 74.9299 0)
+      (effects (font (size 1.27 1.27)) (justify left))
+    )
+    (property "Footprint" "XDCR_COM-09032" (id 2) (at 275.59 72.39 0)
+      (effects (font (size 1.27 1.27)) (justify bottom) hide)
+    )
+    (property "Datasheet" "" (id 3) (at 275.59 72.39 0)
+      (effects (font (size 1.27 1.27)) hide)
+    )
+    (property "MAXIMUM_PACKAGE_HEIGHT" "30.1mm" (id 4) (at 275.59 72.39 0)
+      (effects (font (size 1.27 1.27)) (justify bottom) hide)
+    )
+    (property "PARTREV" "N/A" (id 5) (at 275.59 72.39 0)
+      (effects (font (size 1.27 1.27)) (justify bottom) hide)
+    )
+    (property "STANDARD" "Manufacturer Recommendations" (id 6) (at 275.59 72.39 0)
+      (effects (font (size 1.27 1.27)) (justify bottom) hide)
+    )
+    (property "MANUFACTURER" "SparkFun Electronics" (id 7) (at 275.59 72.39 0)
+      (effects (font (size 1.27 1.27)) (justify bottom) hide)
+    )
+    (pin "B1A")
+    (pin "B2A")
+    (pin "H1")
+    (pin "H2")
+    (pin "H3")
+    (pin "S1")
+    (pin "S2")
+    (pin "S3")
+    (pin "S4")
+    (pin "V1")
+    (pin "V2")
+    (pin "V3")
+  )
   (symbol (lib_id "Connector:USB_B_Mini") (at 208.28 30.48 0) (mirror y) (unit 1)
     (in_bom yes) (on_board yes) (fields_autoplaced)
@@
       (reference "#PWR?") (unit 1) (value "+3.3V") (footprint "")
     )
+    (path "/19143aae-1051-4625-93fe-0e7e3a343a81"
+      (reference "#PWR?") (unit 1) (value "+3.3V") (footprint "")
+    )
     (path "/19ce6091-bf02-41f5-bdc8-e70392f65043"
       (reference "#PWR?") (unit 1) (value "+3.3V") (footprint "")
@@
       (reference "#PWR?") (unit 1) (value "+3.3V") (footprint "")
     )
+    (path "/93ff3b7c-360c-4a20-ac2e-56dc47734d21"
+      (reference "#PWR?") (unit 1) (value "GND") (footprint "")
+    )
     (path "/a8042f04-c07d-4d51-8f79-a5e836d8ad8c"
       (reference "#PWR?") (unit 1) (value "GND") (footprint "")
@@
       (reference "U?") (unit 1) (value "XC6206PxxxMR") (footprint "Package_TO_SOT_SMD:SOT-23")
     )
-  )
+    (path "/e7de9b2e-d01f-464d-888d-e36770a0f879"
+      (reference "U?") (unit 1) (value "COM-09032") (footprint "XDCR_COM-09032")
+    )
+  )

Commit message: I think schematic is done...
Parts:
- added JS2: COM-09032, COM-09032:XDCR_COM-09032, symbol COM-09032:COM-09032
- C1: renamed from C?; footprint (none) -> Button_Switch_SMD:Nidec_Copal_SH-7010A
- JS1: renamed from U?; footprint XDCR_COM-09032 -> COM-09032:XDCR_COM-09032
- SW1, SW10, SW11, SW12, SW2, SW3, SW4, SW5, SW6, SW7, SW8, SW9: footprint (none) -> Button_Switch_SMD:SW_Tactile_SPST_NO_Straight_CK_PTS636Sx25SMTRLFS
- gave numbers to parts that had none: 12
Connections:
- net +3V3: now also JS2.H1 (H+), JS2.V1 (V+)
- net GND: now also JS1.B2A (SEL-), JS2.B2A (SEL-), JS2.H3 (H-), JS2.V3 (V-)
- net PC1: now also MCU1.16 (PC1); no longer MCU1.15 (PC0)
- net SEL1: now reaches JS1.B1A (SEL+)
- net X1: now reaches JS1.H2 (H)
- net Y1: now reaches JS1.V2 (V)
- new net: JS2.S1 (SHIELD), JS2.S2 (SHIELD), JS2.S3 (SHIELD), JS2.S4 (SHIELD)
- new net SEL2: JS2.B1A (SEL+)
- new net X2: JS2.H2 (H)
- new net Y2: JS2.V2 (V)
Other:
- moved on the sheet: J2, JS1

Commit message: assigning footprints
Parts:
- C1: footprint Button_Switch_SMD:Nidec_Copal_SH-7010A -> Button_Switch_THT:SW_Tactile_Straight_KSA0Axx1LFTR
- C3, C4, C5, C6, C7: footprint (none) -> Capacitor_THT:C_Rect_L4.6mm_W2.0mm_P2.50mm_MKS02_FKP02
- FB1: footprint (none) -> Inductor_SMD:L_0603_1608Metric
- R1: footprint (none) -> Resistor_THT:R_Axial_DIN0207_L6.3mm_D2.5mm_P10.16mm_Horizontal
- SW1, SW10, SW11, SW12, SW2, SW3, SW4, SW5, SW6, SW7, SW8, SW9: footprint Button_Switch_SMD:SW_Tactile_SPST_NO_Straight_CK_PTS636Sx25SMTRLFS -> Button_Switch_THT:SW_Tactile_Straight_KSA0Axx1LFTR

Commit message: Finished Footprints
Parts:
- removed J1: USB_B_Mini, symbol Connector:USB_B_Mini
- added C8, C9: C, Capacitor_SMD:C_0805_2012Metric, symbol Device:C
- added J1: USB_B_Micro, Connector_USB:USB_Micro-B_Wuerth_629105150521, symbol Connector:USB_B_Micro
- added L1: L, Inductor_SMD:L_0402_1005Metric, symbol Device:L
- C1: footprint Button_Switch_THT:SW_Tactile_Straight_KSA0Axx1LFTR -> Capacitor_SMD:C_0805_2012Metric
- C2: footprint (none) -> Capacitor_SMD:C_0805_2012Metric
- C3: value C -> 4u7; footprint Capacitor_THT:C_Rect_L4.6mm_W2.0mm_P2.50mm_MKS02_FKP02 -> Capacitor_SMD:C_0805_2012Metric
- C4, C5, C6, C7: value C -> 100n; footprint Capacitor_THT:C_Rect_L4.6mm_W2.0mm_P2.50mm_MKS02_FKP02 -> Capacitor_SMD:C_0805_2012Metric
- D1: footprint (none) -> Diode_SMD:D_0603_1608Metric
- J2: footprint (none) -> Connector_PinHeader_2.54mm:PinHeader_1x04_P2.54mm_Vertical
- R1: footprint Resistor_THT:R_Axial_DIN0207_L6.3mm_D2.5mm_P10.16mm_Horizontal -> Resistor_SMD:R_0805_2012Metric
Connections:
- net +3.3VA: now also C8.1, C9.1, L1.2
- net +3V3: now also L1.1
- net +5V: now also J1.1 (VBUS)
- net GND: now also C8.2, C9.2, J1.5 (GND)
- net USB_DM: now also J1.2 (D-)
- net USB_DP: now also J1.3 (D+)
