File: controller_pcb/controller_pcb/controller_pcb.kicad_pcb (KiCad board)
At the start: 2 copper layers, 34 parts, among them J1 USB_B_Micro, Y1 8MHz

Commit message: added the easy routes lol
Parts:
- turned CONV1 to 180 degrees
- turned FB1 to 180 degrees
Routing:
- net +3V3: track 0.00 -> 264.4 mm
- net Net-(JS2-PadS1): track 0.00 -> 42.9 mm
- net Net-(JS1-PadS1): track 0.00 -> 42.9 mm
- net +5V: track 50.9 -> 17.3 mm
- net +3.3VA: track 0.00 -> 19.0 mm
- net Net-(MCU1-Pad12): track 2.27 -> 19.7 mm
- net VCC: track 0.00 -> 17.3 mm
- net Net-(D1-Pad1): track 0.00 -> 11.6 mm
- net Net-(MCU1-Pad13): track 0.00 -> 11.3 mm
- net USB_DM: track 80.6 -> 86.3 mm
- net (no net): vias 40 -> 32
